Commit message: Added ur10 to robot urdf

File: cob_hardware_config/raw3-4/urdf/raw3-4.urdf.xacro (robot description, xacro)
@@ -15,7 +15,12 @@
   <!-- generic simulator_gazebo plugins for starting mechanism control, ros time, ros battery -->
   <include filename="$(find cob_description)/gazebo/gazebo.urdf.xacro" />
+  <!-- ur_arm -->
+  <include filename="$(find raw_description)/urdf/ur_arm/ur10_arm.urdf.xacro" />
   <xacro:raw_base name="base"/>
   <xacro:tower_asymetric name="tower" parent="base_link">
       <origin xyz="${tower_x} ${tower_y} ${tower_z}" rpy="${tower_roll} ${tower_pitch} ${tower_yaw}" />
   </xacro:tower_asymetric>
+  <xacro:cob_ur10 name="arm" parent="base_link">
+      <origin xyz="${arm_x} ${arm_y} ${arm_z}" rpy="${arm_roll} ${arm_pitch} ${arm_yaw}" />
+  </xacro:cob_ur10>
 </robot>

Commit message: Added cover plate to urdf

File: cob_hardware_config/raw3-4/urdf/raw3-4.urdf.xacro (robot description, xacro)
@@ -24,3 +24,21 @@
       <origin xyz="${arm_x} ${arm_y} ${arm_z}" rpy="${arm_roll} ${arm_pitch} ${arm_yaw}" />
   </xacro:cob_ur10>
+  <!-- additional cover plane -->
+  <link name="cover">
+    <visual>
+      <geometry>
+        <box size="0.725 0.568 .02"/>
+      </geometry>
+    </visual>
+    <collision>
+      <geometry>
+        <box size="0.725 0.568 .02"/>
+      </geometry>
+    </collision>
+  </link>
+  <joint name="base_to_cover" type="fixed">
+       <parent link="base_link"/>
+       <child link="cover"/>
+       <origin xyz="-0.1475 0 0.48"/>
+  </joint>
 </robot>

Commit message: Update raw3-4.urdf.xacro

File: cob_hardware_config/raw3-4/urdf/raw3-4.urdf.xacro (robot description, xacro)
@@ -24,4 +24,10 @@
       <origin xyz="${arm_x} ${arm_y} ${arm_z}" rpy="${arm_roll} ${arm_pitch} ${arm_yaw}" />
   </xacro:cob_ur10>
+   <!-- mount the arm to the robot
+  <joint name="arm_base_joint" type="fixed" >
+      <origin xyz="${arm_x} ${arm_y} ${arm_z}" rpy="${arm_roll} ${arm_pitch} ${arm_yaw}" />
+      <parent link="base_link" />
+      <child link="arm_base_link" />
+  </joint>
   <!-- additional cover plane -->
   <link name="cover">

Commit message: changes on urdf and config

File: cob_hardware_config/raw3-4/urdf/raw3-4.urdf.xacro (robot description, xacro)
@@ -17,4 +17,6 @@
   <!-- ur_arm -->
   <include filename="$(find raw_description)/urdf/ur_arm/ur10_arm.urdf.xacro" />
+  <!-- robotiq gripper -->
+  <include filename="$(find robotiq_description)/urdf/s-model/s-model.urdf.xacro" />
   <xacro:raw_base name="base"/>
   <xacro:tower_asymetric name="tower" parent="base_link">
@@ -24,10 +26,4 @@
       <origin xyz="${arm_x} ${arm_y} ${arm_z}" rpy="${arm_roll} ${arm_pitch} ${arm_yaw}" />
   </xacro:cob_ur10>
-   <!-- mount the arm to the robot
-  <joint name="arm_base_joint" type="fixed" >
-      <origin xyz="${arm_x} ${arm_y} ${arm_z}" rpy="${arm_roll} ${arm_pitch} ${arm_yaw}" />
-      <parent link="base_link" />
-      <child link="arm_base_link" />
-  </joint>
   <!-- additional cover plane -->
   <link name="cover">
@@ -36,4 +32,7 @@
         <box size="0.725 0.568 .02"/>
       </geometry>
+      <material name="grey">
+  	<color rgba="0.8 0.8 0.8 1"/>
+      </material>
     </visual>
     <collision>
@@ -48,3 +47,18 @@
        <origin xyz="-0.1475 0 0.48"/>
   </joint>
+  <link name="quick_changer_link"/>
+  <joint name="changer_to_ee" type="fixed">
+       <parent link="arm_ee_link"/>
+       <child link="quick_changer_link"/>
+       <origin xyz="0.04 0 0" rpy="1.57 -0.45 1.57"/>
+  </joint>
+  <link name="tool_cam_link"/>
+  <joint name="cam_to_changer" type="fixed">
+       <parent link="quick_changer_link"/>
+       <child link="tool_cam_link"/>
+       <origin xyz="0 0 0.095" rpy="0.0 0.0 0.0"/>
+  </joint>
+  <!--xacro:s-model_mesh prefix="gripper" parent="arm_ee_link">
+       <origin xyz="0.15 0 0" rpy="1.57 0.0 1.57"/>
+  </xacro:s-model_mesh-->
 </robot>
